File: final.kicad_sch (KiCad schematic)
At the start: 25 parts, among them J1 Conn_02x16_Odd_Even, J3 USB_C_Receptacle_USB2.0_14P, SW1 SW_Push, U2 INA219AxD, U3 BQ25601, U4 CH224K

Commit message: to resego
Parts:
- removed C10: 100nF, symbol Device:C_Small
- removed C4: 10uF, Capacitor_SMD:CP_Elec_3x5.3, symbol Device:C_Small
- removed C5: 4.7nF, symbol Device:C_Small
- removed C8: 10uF, symbol Device:C_Small
- removed C9: 1uF, symbol Device:C_Small
- removed D1: D_Zener_Filled, symbol Device:D_Zener_Filled
- removed D3: LED_Filled, symbol Device:LED_Filled
- removed J3: USB_C_Receptacle_USB2.0_14P, symbol Connector:USB_C_Receptacle_USB2.0_14P
- removed R10: 10K, symbol Device:R_Small_US
- removed R11: 1k, symbol Device:R_Small_US
- removed R12: 1M, symbol Device:R_Small_US
- removed R8, R9: 2.2k, symbol Device:R_Small_US
- removed SW1: SW_Push, symbol Switch:SW_Push
- removed U3: BQ25601, Package_DFN_QFN:Texas_S-PWQFN-N24_EP2.7x2.7mm_ThermalVias, symbol Battery_Management:BQ25601
- removed U4: CH224K, Package_SO:SSOP-10-1EP_3.9x4.9mm_P1mm_EP2.1x3.3mm, symbol Interface_USB:CH224K
- added C1: 4.7nF, Capacitor_SMD:CP_Elec_3x5.3, symbol Device:C_Small
- added C2: 1uF, symbol Device:C_Small
- added J3: Conn_01x02_Pin, symbol Connector:Conn_01x02_Pin
- added Q1: NMOS, symbol Simulation_SPICE:NMOS
- added R2: 2k, Resistor_SMD:R_0201_0603Metric_Pad0.64x0.40mm_HandSolder, symbol Device:R_Small_US
- added R3: 3k, Resistor_SMD:R_0201_0603Metric_Pad0.64x0.40mm_HandSolder, symbol Device:R_Small_US
- added TP3, TP4: TestPoint, TestPoint:TestPoint_Pad_1.0x1.0mm, symbol Connector:TestPoint
- added U1: MCP73812T-420I-OT, Package_TO_SOT_SMD:SOT-23-5, symbol Battery_Management:MCP73812T-420I-OT
- added U3: HUSB237-AA001-DN06R, Resistor_SMD:R_0201_0603Metric, symbol kutlwano:HUSB237-AA001-DN06R
- added USBC1: USB 3.1 C 6PF, symbol New_Library:USB 3.1 C 6PF
- C3: value 1uF -> 4.7nF
- J1: now not fitted
- R1: footprint (none) -> Resistor_SMD:R_0201_0603Metric
- R4, R5: footprint (none) -> Resistor_SMD:R_0201_0603Metric_Pad0.64x0.40mm_HandSolder
- R6: value R_Small_US -> 75R
- TP1, TP2: footprint (none) -> TestPoint:TestPoint_Pad_1.0x1.0mm
Connections:
- net +9V: now also C2.1, U3.2 (VUSB), USBC1.A9 (VBUS), USBC1.B9 (VBUS)
- net GND: now also R6.2, C1.2, C2.2, J3.1 (Pin_1), Q1.3 (S), U3.7 (GND), USBC1.A12 (GND), USBC1.B12 (GND); no longer C3.2
- net VBAT: no longer R6.1
- new net: C1.1, J3.2 (Pin_2), U1.3 (V_{BAT})
- new net: Q1.1 (D), R2.2, R3.1, TP3.1
- new net: R2.1, U1.5 (PROG)
- new net: U3.1 (CC1), USBC1.A5 (CC1)
- new net: U3.6 (CC2), USBC1.B5 (CC2)
- new net: R3.2, U1.2 (V_{SS})
- new net: C3.2, TP4.1, U1.1 (CE), U1.4 (V_{DD})
- new net: R6.1, U3.3 (VSET)
- new net FAST CHARGE PIN: Q1.2 (G)
- no-connect marks 7 -> 6
